File: hardware/shannon/kicad/shannon.kicad_pcb (KiCad board)
At the start: 2 copper layers, 133.2 x 95 mm, 40 parts

Commit message: shannon PCB fixes
Routing:
- net P3: track 122.8 -> 134.8 mm, vias 0 -> 5
- net P4: track 105.8 -> 117.8 mm, vias 0 -> 5
- net P2: track 145.5 -> 155.1 mm, vias 0 -> 5
- net P10: track 104.1 -> 111.3 mm, vias 0 -> 3
- net ring_top: track 32.7 -> 35.1 mm, vias 1 -> 2
- net middle_home: track 32.7 -> 35.1 mm, vias 1 -> 2
- net inner_default: track 32.7 -> 35.1 mm, vias 1 -> 2
- net ring_home: track 32.7 -> 35.1 mm, vias 1 -> 2
- net middle_top: track 32.7 -> 35.1 mm, vias 1 -> 2
- net index_home: track 32.7 -> 35.1 mm, vias 1 -> 2
- net index_bottom: track 32.7 -> 35.1 mm, vias 1 -> 2
- net inner_bottom: track 32.7 -> 35.1 mm, vias 1 -> 2
- net ring_bottom: track 32.7 -> 35.1 mm, vias 1 -> 2
- net middle_bottom: track 32.7 -> 35.1 mm, vias 1 -> 2
- net pinky_top: track 32.7 -> 35.1 mm, vias 1 -> 2
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Other:
- outline, holes or cut-outs redrawn
